File: Eagle/Linear Sensor/v1/v1.brd (EAGLE design)
At the start: 63.5 x 35.8 mm, 43 parts, among them CON1 SPI, IC1 REG1117, Q1 BSP613P, X3 16MHz, X4 MINI-USB-SCHIELD-32005-201

Commit message: Update linear sensor
Parts:
- moved C10 39.4 mm to (41.9, 3.81)
- moved C12 33.0 mm to (39.4, 3.81)
Changed lines of the file:
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@@
 <element name="C11" library="rcl" package="C1206" value="100nF" x="35.56" y="10.16" rot="R270"/>
 <element name="CON1" library="lpatiny" package="TC2030-MCP-NL" value="SPI" x="12.7" y="12.7" rot="MR90"/>
-<element name="C10" library="rcl" package="C1206" value="10uF" x="2.54" y="3.81" rot="MR90"/>
+<element name="C10" library="rcl" package="C1206" value="10uF" x="41.91" y="3.81" rot="MR90"/>
 <element name="D2" library="lpatiny" package="LED-1206" value="1N581D1206" x="48.26" y="3.81" rot="MR270"/>
 <element name="LED4" library="led" package="CHIP-LED0805" value="RED" x="52.07" y="17.78" rot="R270"/>
 <element name="RL4" library="resistor" package="R0805" value="1K" x="48.26" y="5.08" rot="R90"/>
 <element name="D3" library="lpatiny" package="LED-1206" value="1N581D1206" x="50.8" y="3.81" rot="MR270"/>
-<element name="C12" library="rcl" package="C1206" value="100nF" x="6.35" y="3.81" rot="MR270"/>
+<element name="C12" library="rcl" package="C1206" value="100nF" x="39.37" y="3.81" rot="MR270"/>
 <element name="D4" library="lpatiny" package="LED-1206" value="1N581D1206" x="45.72" y="3.81" rot="MR270"/>
 <element name="RL1" library="rcl" package="R0805" value="1K" x="12.7" y="24.13" rot="MR180"/>
@@
 <wire x1="43.18" y1="16.64" x2="45.72" y2="16.64" width="0" layer="19" extent="16-16"/>
 <wire x1="40.9194" y1="10.8204" x2="43.18" y2="16.64" width="0" layer="19" extent="1-16"/>
-<wire x1="35.56" y1="8.76" x2="40.9194" y2="10.8204" width="0" layer="19" extent="1-1"/>
+<wire x1="41.91" y1="5.21" x2="40.9194" y2="10.8204" width="0" layer="19" extent="1-16"/>
+<wire x1="39.37" y1="5.21" x2="41.91" y2="5.21" width="0" layer="19" extent="16-16"/>
+<wire x1="45.72" y1="6.13" x2="41.91" y2="5.21" width="0" layer="19" extent="1-16"/>
+<wire x1="35.56" y1="8.76" x2="39.37" y2="5.21" width="0" layer="19" extent="1-16"/>
 <wire x1="29.93" y1="10.82" x2="35.56" y2="8.76" width="0" layer="19" extent="1-1"/>
 <wire x1="28.3337" y1="12.065" x2="29.93" y2="10.82" width="0" layer="19" extent="1-16"/>
 <wire x1="24.93" y1="13.42" x2="28.3337" y2="12.065" width="0" layer="19" extent="1-16"/>
 <wire x1="29.93" y1="4.42" x2="29.93" y2="10.82" width="0" layer="19" extent="1-1"/>
-<wire x1="45.72" y1="6.13" x2="40.9194" y2="10.8204" width="0" layer="19" extent="1-1"/>
 <wire x1="21.46" y1="20.32" x2="24.93" y2="13.42" width="0" layer="19" extent="1-1"/>
 <wire x1="19.05" y1="25.27" x2="21.46" y2="20.32" width="0" layer="19" extent="1-16"/>
@@
 <wire x1="2.2225" y1="13.0175" x2="2.54" y2="14.29" width="0" layer="19" extent="1-16"/>
 <wire x1="3.68" y1="7.62" x2="2.2225" y2="13.0175" width="0" layer="19" extent="1-16"/>
-<wire x1="2.54" y1="5.21" x2="3.68" y2="7.62" width="0" layer="19" extent="1-16"/>
-<wire x1="3.68" y1="2.54" x2="2.54" y2="5.21" width="0" layer="19" extent="1-16"/>
-<wire x1="6.35" y1="5.21" x2="3.68" y2="7.62" width="0" layer="19" extent="1-16"/>
+<wire x1="3.68" y1="2.54" x2="3.68" y2="7.62" width="0" layer="19" extent="1-1"/>
 </signal>
 <signal name="SCK">
@@
 <contactref element="U$4" pad="4"/>
 <contactref element="R24" pad="1"/>
+<wire x1="11.75" y1="29.21" x2="20.45" y2="25.4" width="0" layer="19" extent="1-16"/>
 <wire x1="25.73" y1="13.42" x2="20.45" y2="25.4" width="0" layer="19" extent="1-1"/>
-<wire x1="11.75" y1="29.21" x2="20.45" y2="25.4" width="0" layer="19" extent="1-16"/>
 </signal>
 <signal name="D11*">
@@
 <contactref element="U$4" pad="27"/>
 <contactref element="Q1" pad="1"/>
-<wire x1="23.33" y1="1.82" x2="49.759" y2="8.331" width="0" layer="19" extent="1-16"/>
+<wire x1="23.33" y1="1.82" x2="49.759" y2="8.331" width="0" layer="19" extent="1-1"/>
 </signal>
 <signal name="D10*">
@@
 <contactref element="D5" pad="A"/>
 <contactref element="U$1" pad="SI"/>
-<wire x1="32.868" y1="7.62" x2="24.36" y2="20.32" width="0" layer="19" extent="16-16"/>
-<wire x1="20.2438" y1="12.065" x2="32.868" y2="7.62" width="0" layer="19" extent="16-16"/>
+<wire x1="20.2438" y1="12.065" x2="24.36" y2="20.32" width="0" layer="19" extent="16-16"/>
+<wire x1="32.868" y1="7.62" x2="20.2438" y2="12.065" width="0" layer="19" extent="16-16"/>
 </signal>
 <signal name="N$10">
@@
 <contactref element="U$2" pad="1"/>
 <contactref element="C4" pad="2"/>
-<wire x1="48.13" y1="27.94" x2="44.45" y2="24.13" width="0" layer="19" extent="1-1"/>
-<wire x1="45.72" y1="13.84" x2="48.13" y2="27.94" width="0" layer="19" extent="1-16"/>
+<wire x1="44.45" y1="24.13" x2="48.13" y2="27.94" width="0" layer="19" extent="16-16"/>
+<wire x1="45.72" y1="13.84" x2="44.45" y2="24.13" width="0" layer="19" extent="16-16"/>
 <wire x1="45.4914" y1="10.8204" x2="45.72" y2="13.84" width="0" layer="19" extent="1-16"/>
 <wire x1="48.26" y1="4.23" x2="45.4914" y2="10.8204" width="0" layer="19" extent="1-1"/>
@@
 <wire x1="50.8" y1="2.31" x2="48.26" y2="2.31" width="0" layer="19" extent="16-16"/>
 <wire x1="45.72" y1="2.31" x2="48.26" y2="2.31" width="0" layer="19" extent="16-16"/>
-<wire x1="29.93" y1="11.62" x2="45.4914" y2="10.8204" width="0" layer="19" extent="1-1"/>
+<wire x1="41.91" y1="2.41" x2="45.72" y2="2.31" width="0" layer="19" extent="16-16"/>
+<wire x1="39.37" y1="2.41" x2="41.91" y2="2.41" width="0" layer="19" extent="16-16"/>
+<wire x1="29.93" y1="3.62" x2="39.37" y2="2.41" width="0" layer="19" extent="1-16"/>
+<wire x1="29.93" y1="11.62" x2="29.93" y2="3.62" width="0" layer="19" extent="1-1"/>
 <wire x1="27.33" y1="13.42" x2="29.93" y2="11.62" width="0" layer="19" extent="1-1"/>
-<wire x1="29.93" y1="3.62" x2="29.93" y2="11.62" width="0" layer="19" extent="1-1"/>
 <wire x1="20.93" y1="1.82" x2="29.93" y2="3.62" width="0" layer="19" extent="1-1"/>
 <wire x1="18.33" y1="10.02" x2="20.93" y2="1.82" width="0" layer="19" extent="1-1"/>
 <wire x1="7.62" y1="14.29" x2="18.33" y2="10.02" width="0" layer="19" extent="1-1"/>
-<wire x1="6.35" y1="2.41" x2="7.62" y2="14.29" width="0" layer="19" extent="1-16"/>
-<wire x1="2.54" y1="2.41" x2="6.35" y2="2.41" width="0" layer="19" extent="16-16"/>
 </signal>
 <signal name="D8*">
